Commit message: fix numerical precision

File: assets/maze_boundary.urdf (robot description, URDF)
Before this commit: robot maze_boundary, 5 links, 4 joints
Joints:
- joint bottom_left_corner: origin xyz=5 5 0 rpy=0 0 1.5708 -> xyz=5 5 0 rpy=0 0 1.5707963268
- joint bottom_right_corner: origin xyz=5 5 0 rpy=0 0 1.5708 -> xyz=5 5 0 rpy=0 0 1.5707963268
- joint top_left_corner: origin xyz=5 5 0 rpy=0 0 1.5708 -> xyz=5 5 0 rpy=0 0 1.5707963268
